File: hardware/RFWBBoard/RFWBBoard.brd (EAGLE design)
At the start: 90.2 x 56 mm, 84 parts, among them IC1 24LC025ST, J1 CON-71742-2184-BOT, M1 MOUNT-HOLE3.3, M2 MOUNT-HOLE3.3, M3 MOUNT-HOLE3.3, M4 MOUNT-HOLE3.3, U1 MAX2830IPC-7351, U2 LDB212G4010C-001, U3 LDB212G4010C-001, U4 AD8132MSOP8, U5 AD8132MSOP8, U6 AD8132MSOP8, U7 AD8132MSOP8, X1 LTI-SASF54GT, X2 LTI-SASF54GT, X4 LTI-SASF54GT, X5 LTI-SASF54GT, X6 LTI-SASF54GT, X7 LTI-SASF54GT

Commit message: - Added info text on bottom
Other:
- board text added: "RF Board"
- board text added: "Wideband 2.4 GHz/Baseband module"
- board text added: "for the Marmote platform"
- board text added: "http://marmote.googlecode.com"
Changed lines of the file:
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@@
 <layers>
 <layer number="1" name="Top" color="4" fill="1" visible="yes" active="yes"/>
-<layer number="2" name="Route2" color="14" fill="1" visible="no" active="yes"/>
-<layer number="3" name="Route3" color="4" fill="1" visible="no" active="yes"/>
+<layer number="2" name="Route2" color="14" fill="1" visible="yes" active="yes"/>
+<layer number="3" name="Route3" color="4" fill="1" visible="yes" active="yes"/>
 <layer number="14" name="Route14" color="1" fill="6" visible="no" active="no"/>
 <layer number="15" name="Route15" color="4" fill="6" visible="no" active="no"/>
-<layer number="16" name="Bottom" color="14" fill="1" visible="no" active="yes"/>
+<layer number="16" name="Bottom" color="14" fill="1" visible="yes" active="yes"/>
 <layer number="17" name="Pads" color="2" fill="1" visible="yes" active="yes"/>
-<layer number="18" name="Vias" color="2" fill="1" visible="no" active="yes"/>
+<layer number="18" name="Vias" color="2" fill="1" visible="yes" active="yes"/>
 <layer number="19" name="Unrouted" color="6" fill="1" visible="yes" active="yes"/>
 <layer number="20" name="Dimension" color="15" fill="1" visible="yes" active="yes"/>
@@
 <layer number="37" name="tTest" color="7" fill="1" visible="no" active="yes"/>
 <layer number="38" name="bTest" color="7" fill="1" visible="no" active="yes"/>
-<layer number="39" name="tKeepout" color="4" fill="11" visible="yes" active="yes"/>
+<layer number="39" name="tKeepout" color="4" fill="11" visible="no" active="yes"/>
 <layer number="40" name="bKeepout" color="1" fill="11" visible="yes" active="yes"/>
 <layer number="41" name="tRestrict" color="4" fill="10" visible="yes" active="yes"/>
 <layer number="42" name="bRestrict" color="1" fill="10" visible="yes" active="yes"/>
 <layer number="43" name="vRestrict" color="2" fill="10" visible="no" active="yes"/>
-<layer number="44" name="Drills" color="7" fill="1" visible="no" active="yes"/>
+<layer number="44" name="Drills" color="7" fill="1" visible="yes" active="yes"/>
 <layer number="45" name="Holes" color="7" fill="1" visible="yes" active="yes"/>
 <layer number="46" name="Milling" color="3" fill="1" visible="no" active="yes"/>
@@
 <layer number="50" name="dxf" color="7" fill="1" visible="no" active="yes"/>
 <layer number="51" name="tDocu" color="7" fill="1" visible="yes" active="yes"/>
-<layer number="52" name="bDocu" color="7" fill="1" visible="no" active="yes"/>
+<layer number="52" name="bDocu" color="7" fill="1" visible="yes" active="yes"/>
 <layer number="53" name="tGND_GNDA" color="7" fill="9" visible="no" active="no"/>
 <layer number="54" name="bGND_GNDA" color="1" fill="9" visible="no" active="no"/>
@@
 <wire x1="52" y1="54" x2="52" y2="50" width="0.4064" layer="51"/>
 <wire x1="52" y1="50" x2="37" y2="50" width="0.4064" layer="51"/>
+<wire x1="26" y1="36" x2="26" y2="24" width="0.2032" layer="52"/>
+<wire x1="26" y1="24" x2="64" y2="24" width="0.2032" layer="52"/>
+<wire x1="64" y1="24" x2="64" y2="36" width="0.2032" layer="52"/>
+<wire x1="64" y1="36" x2="26" y2="36" width="0.2032" layer="52"/>
+<text x="51" y="33" size="1.778" layer="52" font="vector" rot="MR0">RF Board</text>
+<text x="63" y="30" size="1.27" layer="52" font="vector" rot="MR0">Wideband 2.4 GHz/Baseband module</text>
+<text x="57.75" y="27.75" size="1.27" layer="52" font="vector" rot="MR0">for the Marmote platform</text>
+<text x="60.25" y="25.25" size="1.27" layer="52" font="vector" rot="MR0">http://marmote.googlecode.com</text>
 </plain>
 <attributes>
