File: hardware/M6-RF315/M6RF-315.brd (EAGLE design)
At the start: 90 x 56 mm, 38 parts, among them J1 CON-71439-2164, M1 MOUNT-HOLE3.3, M2 MOUNT-HOLE3.3, M3 MOUNT-HOLE3.3, M4 MOUNT-HOLE3.3, M5 FIDUCIAL1X2, M6 FIDUCIAL1X2, M7 FIDUCIAL1X2, M8 FIDUCIAL1X2, U1 CC1101RTKR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

Commit message: Modified GPIO-serial data connection, added LEDs, updated and cleaned up the library, defined antenna circuit component values and added datasheet..
Parts:
- removed X2: NX3225GA, M6-RF315:NX3225GA
- added J2: CON-SMA-VERT, M6-RF315:SMA-VERT
- added LED1, LED2: (no value), M6-RF315:LED0603
- added R3: 500, M6-RF315:R0603
- added R4: 130, M6-RF315:R0603
- C10, C14: value (none) -> 220pF
- C11, C13: value (none) -> 6.8pF
- C12: value (none) -> 12pF
- C9: value (none) -> 6.8 pF
- L1, L2, L4: value (none) -> 33nH
- L3: value (none) -> 18nH
- X1: value CON-SMA -> NX3225GA; device M6-RF315:LTI-SASF54GT -> M6-RF315:NX3225GA
- moved X1 22.6 mm to (50.0, 20.0), turned to 270 degrees
- moved TP1 6.40 mm to (32.0, 14.0)
- moved TP2 1.00 mm to (58.0, 14.0)
Connections:
- removed net I2C1_SCL: J1.14
- removed net I2C1_SDA: J1.16
- removed net N$5: C6.2
- new net N$19: LED2.A, R4.1
- new net PB6: J1.14, LED2.C
- new net PB7: J1.16, LED1.C
- net AGND: now also J2.2; no longer X1.2
- net D3V3: now also R3.2, R4.2
- net DGND: now also C6.2, X1.2, X1.4; no longer X2.2, X2.4
- net GND: now also J2.3, J2.4, J2.5; no longer X1.3, X1.4, X1.5
- net N$1: now also LED1.A, R3.1; no longer J1.34, U1.3
- net N$12: now also J2.1; no longer X1.1
- net N$6: now also X1.1; no longer X2.1
- net N$7: now also X1.3; no longer X2.3
- net PA10: now also TP1.1, U1.6; no longer TP2.1
- net PA9: now also J1.34; no longer TP1.1, U1.6
- net PB4: now also TP2.1, U1.3

Commit message: Started routing.
Parts:
- moved C8 9.15 mm to (50.0, 22.0), turned to 0 degrees
- moved C5 8.68 mm to (46.5, 14.2), turned to 270 degrees
- moved C1 8.49 mm to (39.0, 20.0), turned to 180 degrees
- moved C7 8.46 mm to (52.0, 16.0), turned to 0 degrees
- moved C2 5.10 mm to (54.0, 14.0)
- moved C6 2.71 mm to (49.0, 16.0), turned to 0 degrees
- moved X1 1.00 mm to (50.0, 19.0)
Routing:
- net SPI1_MOSI: track 0.00 -> 10.1 mm, vias 0 -> 1
- net SPI1_SCK: track 0.00 -> 10.1 mm, vias 0 -> 1
- net SPI1_MISO: track 0.00 -> 9.85 mm, vias 0 -> 1
- net PB4: track 0.00 -> 9.23 mm, vias 0 -> 1
- net N$7: track 0.00 -> 6.79 mm
- net N$6: track 0.00 -> 4.37 mm
- net N$4: track 0.00 -> 3.01 mm
- net D3V3: track 0.00 -> 2.41 mm

Commit message: M6-RF315 board 80% routed (9 airwires remaining).
Parts:
- moved LOGO2 53.2 mm to (66.0, 13.0)
- moved U$3 48.0 mm to (14.0, 34.0)
- moved TP1 44.3 mm to (74.0, 28.0)
- moved R4 24.8 mm to (13.8, 29.0), flipped to the bottom, turned to 0 degrees
- moved R3 21.2 mm to (13.8, 27.0), flipped to the bottom, turned to 0 degrees
- moved LED2 20.6 mm to (16.0, 28.0), turned to 0 degrees
- moved LOGO1 18.4 mm to (66.0, 34.0)
- moved TP2 17.2 mm to (68.0, 28.0)
- moved R1 15.8 mm to (38.2, 21.0), turned to 90 degrees
- moved C4 13.3 mm to (40.8, 21.5), turned to 180 degrees
- moved C3 12.9 mm to (41.8, 22.0), flipped to the bottom
- moved LED1 12.1 mm to (22.0, 28.0), turned to 0 degrees
- moved C1 11.0 mm to (50.0, 20.0), flipped to the bottom
- moved C2 9.43 mm to (49.0, 22.0), flipped to the bottom, turned to 180 degrees
- moved LOGO3 5.00 mm to (14.0, 13.0)
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Connections:
- net N$3 renamed RBIAS
- removed net GND: J2.3, J2.4, J2.5
- net AGND: now also J2.3, J2.4, J2.5
Routing:
- net AGND: track 0.00 -> 71.1 mm, vias 0 -> 5
- net D3V3: track 2.41 -> 53.1 mm, vias 0 -> 2
- net A3V3: track 0.00 -> 43.5 mm, vias 0 -> 3
- net PA10: track 0.00 -> 42.7 mm, vias 0 -> 2
- net DGND: track 0.00 -> 38.5 mm, vias 0 -> 7
- net PB6: track 0.00 -> 31.3 mm, vias 0 -> 1
- net PB4: track 9.23 -> 39.6 mm, vias 1 -> 2
- net PB7: track 0.00 -> 26.6 mm, vias 0 -> 1
- net SPI1_NSS: track 0.00 -> 19.2 mm, vias 0 -> 2
- net N$1: track 0.00 -> 10.6 mm, vias 0 -> 1
- net N$12: track 0.00 -> 6.50 mm
- net N$8: track 0.00 -> 6.02 mm
- net N$9: track 0.00 -> 5.72 mm
- net RBIAS: track 0.00 -> 5.17 mm
- net N$10: track 0.00 -> 4.04 mm
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- added copper zone on layer 1, net AGND
- added copper zone on layer 16, net AGND
- added copper zone on layer 1, net DGND
- added copper zone on layer 16, net DGND
Other:
- board text added: "RX"
- board text added: "TX"
