File: hardware/M6-RF315/M6-RF315.sch (EAGLE design)
At the start: 42 parts, among them J1 CON-71439-2164, J2 CON-SMA-VERT, M1 MOUNT-HOLE3.3, M2 MOUNT-HOLE3.3, M3 MOUNT-HOLE3.3, M4 MOUNT-HOLE3.3, M5 FIDUCIAL1X2, M6 FIDUCIAL1X2, M7 FIDUCIAL1X2, M8 FIDUCIAL1X2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

Commit message: Added a BOM file (not finished yet).
Parts:
- C9: value 6.8 pF -> 6.8pF
- renumbered U$3 to LOGO4
Other:
- note removed: "- Route PCB design"
Changed lines of the file:
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@@
 <setting verticaltext="up"/>
 </settings>
-<grid distance="0.1" unitdist="inch" unit="inch" style="lines" multiple="1" display="no" altdistance="0.05" altunitdist="inch" altunit="inch"/>
+<grid distance="0.1" unitdist="inch" unit="inch" style="lines" multiple="1" display="no" altdistance="0.01" altunitdist="inch" altunit="inch"/>
 <layers>
 <layer number="1" name="Top" color="4" fill="1" visible="no" active="no"/>
@@
 <part name="TP2" library="M6-RF315" deviceset="TESTPOINT" device="" technology="-RED"/>
 <part name="R2" library="M6-RF315" deviceset="R" device="0603" value="100k"/>
-<part name="C9" library="M6-RF315" deviceset="C" device="0603" value="6.8 pF">
+<part name="C9" library="M6-RF315" deviceset="C" device="0603" value="6.8pF">
 <attribute name="FUNCTION" value="RF balun/matching capacitor"/>
 </part>
@@
 <part name="U$13" library="M6-RF315" deviceset="AGND" device=""/>
 <part name="U$14" library="M6-RF315" deviceset="AGND" device=""/>
-<part name="U$3" library="M6-RF315" deviceset="LOGO-RADIO-2-600MIL" device="-10MM-CU"/>
+<part name="LOGO4" library="M6-RF315" deviceset="LOGO-RADIO-2-600MIL" device="-10MM-CU"/>
 <part name="X1" library="M6-RF315" deviceset="NX3225GA" device=""/>
 <part name="PORT10" library="M6-RF315" deviceset="PORT5" device=""/>
@@
 <instance part="LOGO2" gate="G$1" x="129.54" y="55.88"/>
 <instance part="LOGO3" gate="G$1" x="78.74" y="55.88"/>
-<instance part="U$3" gate="G$1" x="154.94" y="55.88"/>
+<instance part="LOGO4" gate="G$1" x="154.94" y="55.88"/>
 </instances>
 <busses>
@@
 <text x="101.6" y="81.28" size="2.54" layer="98">TODO:</text>
 <wire x1="96.52" y1="88.9" x2="200.66" y2="88.9" width="0.1524" layer="98"/>
-<wire x1="200.66" y1="88.9" x2="200.66" y2="58.42" width="0.1524" layer="98"/>
-<wire x1="200.66" y1="58.42" x2="96.52" y2="58.42" width="0.1524" layer="98"/>
-<wire x1="96.52" y1="58.42" x2="96.52" y2="88.9" width="0.1524" layer="98"/>
+<wire x1="200.66" y1="88.9" x2="200.66" y2="68.58" width="0.1524" layer="98"/>
+<wire x1="200.66" y1="68.58" x2="96.52" y2="68.58" width="0.1524" layer="98"/>
+<wire x1="96.52" y1="68.58" x2="96.52" y2="88.9" width="0.1524" layer="98"/>
 <text x="83.82" y="109.22" size="1.778" layer="95">SERIAL TX DATA</text>
 <text x="83.82" y="106.68" size="1.778" layer="95">SERIAL RX DATA</text>
-<text x="104.14" y="63.5" size="2.54" layer="98">- Check BOM against CC1101 reference BOM for 315 MHz</text>
+<text x="104.14" y="71.12" size="2.54" layer="98">- Check BOM against CC1101 reference BOM for 315 MHz</text>
 <text x="238.76" y="149.86" size="1.778" layer="97" rot="R270">Digikey: ANT-315-CW-RH-SMA-ND</text>
-<text x="104.14" y="68.58" size="2.54" layer="98">- Create BOM file</text>
-<text x="104.14" y="73.66" size="2.54" layer="98">- Route PCB design</text>
+<text x="104.14" y="76.2" size="2.54" layer="98">- Create BOM file</text>
 <text x="71.12" y="109.22" size="1.778" layer="97">NC</text>
 <text x="71.12" y="106.68" size="1.778" layer="97">NC</text>

Commit message: Finished BOM file for M6-RF315.
Parts:
- L1, L2, L3, L4: device M6-RF315:L0603 -> M6-RF315:L0402
Other:
- note removed: "- Check BOM against CC1101 reference BOM for 315 MHz"
- note removed: "- Create BOM file"
- note removed: "TODO:"
Changed lines of the file:
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@@
 <grid distance="0.1" unitdist="inch" unit="inch" style="lines" multiple="1" display="no" altdistance="0.01" altunitdist="inch" altunit="inch"/>
 <layers>
-<layer number="1" name="Top" color="4" fill="1" visible="no" active="no"/>
-<layer number="2" name="Route2" color="1" fill="3" visible="no" active="no"/>
-<layer number="3" name="Route3" color="4" fill="3" visible="no" active="no"/>
-<layer number="14" name="Route14" color="1" fill="6" visible="no" active="no"/>
-<layer number="15" name="Route15" color="4" fill="6" visible="no" active="no"/>
-<layer number="16" name="Bottom" color="1" fill="1" visible="no" active="no"/>
-<layer number="17" name="Pads" color="2" fill="1" visible="no" active="no"/>
-<layer number="18" name="Vias" color="2" fill="1" visible="no" active="no"/>
-<layer number="19" name="Unrouted" color="6" fill="1" visible="no" active="no"/>
-<layer number="20" name="Dimension" color="15" fill="1" visible="no" active="no"/>
-<layer number="21" name="tPlace" color="7" fill="1" visible="no" active="no"/>
-<layer number="22" name="bPlace" color="7" fill="1" visible="no" active="no"/>
-<layer number="23" name="tOrigins" color="15" fill="1" visible="no" active="no"/>
-<layer number="24" name="bOrigins" color="15" fill="1" visible="no" active="no"/>
-<layer number="25" name="tNames" color="7" fill="1" visible="no" active="no"/>
-<layer number="26" name="bNames" color="7" fill="1" visible="no" active="no"/>
-<layer number="27" name="tValues" color="7" fill="1" visible="no" active="no"/>
-<layer number="28" name="bValues" color="7" fill="1" visible="no" active="no"/>
+<layer number="1" name="Top" color="4" fill="1" visible="yes" active="no"/>
+<layer number="2" name="Route2" color="1" fill="3" visible="yes" active="no"/>
+<layer number="3" name="Route3" color="4" fill="3" visible="yes" active="no"/>
+<layer number="14" name="Route14" color="1" fill="6" visible="yes" active="no"/>
+<layer number="15" name="Route15" color="4" fill="6" visible="yes" active="no"/>
+<layer number="16" name="Bottom" color="1" fill="1" visible="yes" active="no"/>
+<layer number="17" name="Pads" color="2" fill="1" visible="yes" active="no"/>
+<layer number="18" name="Vias" color="2" fill="1" visible="yes" active="no"/>
+<layer number="19" name="Unrouted" color="6" fill="1" visible="yes" active="no"/>
+<layer number="20" name="Dimension" color="15" fill="1" visible="yes" active="no"/>
+<layer number="21" name="tPlace" color="7" fill="1" visible="yes" active="no"/>
+<layer number="22" name="bPlace" color="7" fill="1" visible="yes" active="no"/>
+<layer number="23" name="tOrigins" color="15" fill="1" visible="yes" active="no"/>
+<layer number="24" name="bOrigins" color="15" fill="1" visible="yes" active="no"/>
+<layer number="25" name="tNames" color="7" fill="1" visible="yes" active="no"/>
+<layer number="26" name="bNames" color="7" fill="1" visible="yes" active="no"/>
+<layer number="27" name="tValues" color="7" fill="1" visible="yes" active="no"/>
+<layer number="28" name="bValues" color="7" fill="1" visible="yes" active="no"/>
 <layer number="29" name="tStop" color="7" fill="3" visible="no" active="no"/>
 <layer number="30" name="bStop" color="7" fill="6" visible="no" active="no"/>
@@
 <layer number="35" name="tGlue" color="7" fill="4" visible="no" active="no"/>
 <layer number="36" name="bGlue" color="7" fill="5" visible="no" active="no"/>
-<layer number="37" name="tTest" color="7" fill="1" visible="no" active="no"/>
-<layer number="38" name="bTest" color="7" fill="1" visible="no" active="no"/>
+<layer number="37" name="tTest" color="7" fill="1" visible="yes" active="no"/>
+<layer number="38" name="bTest" color="7" fill="1" visible="yes" active="no"/>
 <layer number="39" name="tKeepout" color="4" fill="11" visible="no" active="no"/>
 <layer number="40" name="bKeepout" color="1" fill="11" visible="no" active="no"/>
@@
 <layer number="44" name="Drills" color="7" fill="1" visible="no" active="no"/>
 <layer number="45" name="Holes" color="7" fill="1" visible="no" active="no"/>
-<layer number="46" name="Milling" color="3" fill="1" visible="no" active="no"/>
-<layer number="47" name="Measures" color="7" fill="1" visible="no" active="no"/>
-<layer number="48" name="Document" color="7" fill="1" visible="no" active="no"/>
-<layer number="49" name="Reference" color="7" fill="1" visible="no" active="no"/>
-<layer number="50" name="dxf" color="7" fill="1" visible="no" active="no"/>
-<layer number="51" name="tDocu" color="7" fill="1" visible="no" active="no"/>
-<layer number="52" name="bDocu" color="7" fill="1" visible="no" active="no"/>
-<layer number="53" name="tGND_GNDA" color="7" fill="9" visible="no" active="no"/>
-<layer number="54" name="bGND_GNDA" color="1" fill="9" visible="no" active="no"/>
-<layer number="56" name="wert" color="7" fill="1" visible="no" active="no"/>
+<layer number="46" name="Milling" color="3" fill="1" visible="yes" active="no"/>
+<layer number="47" name="Measures" color="7" fill="1" visible="yes" active="no"/>
+<layer number="48" name="Document" color="7" fill="1" visible="yes" active="no"/>
+<layer number="49" name="Reference" color="7" fill="1" visible="yes" active="no"/>
+<layer number="50" name="dxf" color="7" fill="1" visible="yes" active="no"/>
+<layer number="51" name="tDocu" color="7" fill="1" visible="yes" active="no"/>
+<layer number="52" name="bDocu" color="7" fill="1" visible="yes" active="no"/>
+<layer number="53" name="tGND_GNDA" color="7" fill="9" visible="yes" active="no"/>
+<layer number="54" name="bGND_GNDA" color="1" fill="9" visible="yes" active="no"/>
+<layer number="56" name="wert" color="7" fill="1" visible="yes" active="no"/>
 <layer number="91" name="Nets" color="2" fill="1" visible="yes" active="yes"/>
 <layer number="92" name="Busses" color="1" fill="1" visible="yes" active="yes"/>
@@
 </part>
 <part name="U$10" library="M6-RF315" deviceset="AGND" device=""/>
-<part name="L1" library="M6-RF315" deviceset="L" device="0603" value="33nH">
+<part name="L1" library="M6-RF315" deviceset="L" device="0402" value="33nH">
 <attribute name="FUNCTION" value="RF balun/matching inductor"/>
 </part>
-<part name="L2" library="M6-RF315" deviceset="L" device="0603" value="33nH">
+<part name="L2" library="M6-RF315" deviceset="L" device="0402" value="33nH">
 <attribute name="FUNCTION" value="RF balun/matching inductor"/>
 </part>
 <part name="U$11" library="M6-RF315" deviceset="DGND" device=""/>
-<part name="L3" library="M6-RF315" deviceset="L" device="0603" value="18nH">
+<part name="L3" library="M6-RF315" deviceset="L" device="0402" value="18nH">
 <attribute name="FUNCTION" value="RF LC filter/matching filter inductor"/>
 </part>
-<part name="L4" library="M6-RF315" deviceset="L" device="0603" value="33nH">
+<part name="L4" library="M6-RF315" deviceset="L" device="0402" value="33nH">
 <attribute name="FUNCTION" value="RF LC filter/matching filter inductor"/>
 </part>
@@
 <text x="33.02" y="55.88" size="2.54" layer="97">South bridge</text>
 <text x="177.8" y="20.32" size="5.08" layer="97">&gt;PAGE2</text>
-<text x="101.6" y="81.28" size="2.54" layer="98">TODO:</text>
-<wire x1="96.52" y1="88.9" x2="200.66" y2="88.9" width="0.1524" layer="98"/>
-<wire x1="200.66" y1="88.9" x2="200.66" y2="68.58" width="0.1524" layer="98"/>
-<wire x1="200.66" y1="68.58" x2="96.52" y2="68.58" width="0.1524" layer="98"/>
-<wire x1="96.52" y1="68.58" x2="96.52" y2="88.9" width="0.1524" layer="98"/>
 <text x="83.82" y="109.22" size="1.778" layer="95">SERIAL TX DATA</text>
 <text x="83.82" y="106.68" size="1.778" layer="95">SERIAL RX DATA</text>
-<text x="104.14" y="71.12" size="2.54" layer="98">- Check BOM against CC1101 reference BOM for 315 MHz</text>
 <text x="238.76" y="149.86" size="1.778" layer="97" rot="R270">Digikey: ANT-315-CW-RH-SMA-ND</text>
-<text x="104.14" y="76.2" size="2.54" layer="98">- Create BOM file</text>
 <text x="71.12" y="109.22" size="1.778" layer="97">NC</text>
 <text x="71.12" y="106.68" size="1.778" layer="97">NC</text>

Commit message: Added exported GERBER files.
Parts:
- LOGO4: value LOGO-RADIO-2-600MIL-10MM-CU -> LOGO-RADIO-3-600MIL-10MM-CU; device M6-RF315:LOGO-RADIO-2-600MIL-10MM-CU -> M6-RF315:LOGO-RADIO-3-600MIL-10MM-CU
Changed lines of the file:
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@@
 <part name="U$13" library="M6-RF315" deviceset="AGND" device=""/>
 <part name="U$14" library="M6-RF315" deviceset="AGND" device=""/>
-<part name="LOGO4" library="M6-RF315" deviceset="LOGO-RADIO-2-600MIL" device="-10MM-CU"/>
+<part name="LOGO4" library="M6-RF315" deviceset="LOGO-RADIO-3-600MIL" device="-10MM-CU"/>
 <part name="X1" library="M6-RF315" deviceset="NX3225GA" device=""/>
 <part name="PORT10" library="M6-RF315" deviceset="PORT5" device=""/>
