File: hardware/BreakoutBoard/BreakoutBoard.brd (EAGLE design)
At the start: 90 x 56 mm, 38 parts, among them J1 CON-71741-2184-TOP, J10 CON-2X3-RASTER, J11 CON-2X3-RASTER, J12 CON-2X3-RASTER, J13 CON-2X4-RASTER, J2 CON-71741-2184-BOT, J3 CON-2X4-RASTER, J4 CON-2X10-RASTER, J5 CON-2X3-RASTER, J6 CON-2X3-RASTER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

Commit message: - Logos - Gerber files - Pick and Place file - Assembly Drawings
Parts:
- removed LOGO2: LOGO-VANDERBILT-600MIL-10MM-AU, Logo:LOGO-VANDERBILT-10MM-GOLD
- removed LOGO3: LOGO-MARMOTE-600MIL-10MM-AU, Logo:LOGO-MARMOTE-10MM-GOLD
- removed LOGO4: LOGO-MAGNIFYING-GLASS-600MIL-10MM-AU, Logo:LOGO-MAGNIFYING-GLASS-10MM-GOLD
- added LOGO5: LOGO-VANDERBILT-600MIL-10MM-SS, Logo:LOGO-VANDERBILT-10MM-SILKSCREEN
- added LOGO6: LOGO-ISIS-600MIL-10MM-SS, Logo:LOGO-ISIS-10MM-SILKSCREEN
- added LOGO7: LOGO-MARMOTE-600MIL-10MM-SS, Logo:LOGO-MARMOTE-10MM-SILKSCREEN
- LOGO1: value LOGO-ISIS-600MIL-10MM-AU -> LOGO-MAGNIFYING-GLASS-600MIL-10MM-SS; device Logo:LOGO-ISIS-10MM-GOLD -> Logo:LOGO-MAGNIFYING-GLASS-10MM-SILKSCREEN
- moved LOGO1 52.9 mm to (64.0, 24.5)
Routing:
- net 1: track 20.5 -> 21.7 mm
- net 2: track 24.0 -> 24.6 mm

Commit message: - Gerber files updated - Assembly files updated - Pick and Place updated - BOM - Schematic
Parts:
- moved TP14 1.56 mm to (86.2, 11.5)
- moved TP11 1.56 mm to (3.80, 11.5)
Changed lines of the file:
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@@
 <layer number="23" name="tOrigins" color="15" fill="1" visible="yes" active="yes"/>
 <layer number="24" name="bOrigins" color="15" fill="1" visible="yes" active="yes"/>
-<layer number="25" name="tNames" color="4" fill="1" visible="yes" active="yes"/>
-<layer number="26" name="bNames" color="1" fill="1" visible="yes" active="yes"/>
-<layer number="27" name="tValues" color="7" fill="1" visible="yes" active="yes"/>
-<layer number="28" name="bValues" color="7" fill="1" visible="yes" active="yes"/>
+<layer number="25" name="tNames" color="4" fill="1" visible="no" active="yes"/>
+<layer number="26" name="bNames" color="1" fill="1" visible="no" active="yes"/>
+<layer number="27" name="tValues" color="7" fill="1" visible="no" active="yes"/>
+<layer number="28" name="bValues" color="7" fill="1" visible="no" active="yes"/>
 <layer number="29" name="tStop" color="7" fill="3" visible="yes" active="yes"/>
 <layer number="30" name="bStop" color="7" fill="6" visible="yes" active="yes"/>
@@
 <text x="3" y="50" size="1.27" layer="21" font="vector" rot="R90">DGND</text>
 <text x="88" y="50" size="1.27" layer="21" font="vector" rot="R90">AGND</text>
-<text x="3" y="8.3" size="1.27" layer="21" font="vector" rot="R90">DGND</text>
-<text x="88" y="8.4" size="1.27" layer="21" font="vector" rot="R90">AGND</text>
+<text x="2" y="9.3" size="1.27" layer="21" font="vector" rot="R90">DGND</text>
+<text x="89" y="9.3" size="1.27" layer="21" font="vector" rot="R90">AGND</text>
 <text x="26.7" y="54" size="1.27" layer="21" font="vector">A1V5</text>
 <text x="32" y="54" size="1.27" layer="21" font="vector">A3V3</text>
@@
 <attribute name="MPN" value="5121" x="31.2" y="65" size="1.778" layer="27" display="off"/>
 </element>
-<element name="TP11" library="BreakoutBoard" package="TESTPOINT" value="TESTPOINT-YELLOW" x="5" y="10.5">
-<attribute name="DIGI-KEY#" value="5009K-ND" x="5" y="10.5" size="1.778" layer="27" display="off"/>
-<attribute name="MF" value="Keystone" x="5" y="10.5" size="1.778" layer="27" display="off"/>
-<attribute name="MPN" value="5009" x="5" y="10.5" size="1.778" layer="27" display="off"/>
-</element>
-<element name="TP14" library="BreakoutBoard" package="TESTPOINT" value="TESTPOINT-YELLOW" x="85" y="10.5">
-<attribute name="DIGI-KEY#" value="5009K-ND" x="85" y="10.5" size="1.778" layer="27" display="off"/>
-<attribute name="MF" value="Keystone" x="85" y="10.5" size="1.778" layer="27" display="off"/>
-<attribute name="MPN" value="5009" x="85" y="10.5" size="1.778" layer="27" display="off"/>
+<element name="TP11" library="BreakoutBoard" package="TESTPOINT" value="TESTPOINT-YELLOW" x="3.8" y="11.5">
+<attribute name="DIGI-KEY#" value="5009K-ND" x="3.8" y="11.5" size="1.778" layer="27" display="off"/>
+<attribute name="MF" value="Keystone" x="3.8" y="11.5" size="1.778" layer="27" display="off"/>
+<attribute name="MPN" value="5009" x="3.8" y="11.5" size="1.778" layer="27" display="off"/>
+</element>
+<element name="TP14" library="BreakoutBoard" package="TESTPOINT" value="TESTPOINT-YELLOW" x="86.2" y="11.5">
+<attribute name="DIGI-KEY#" value="5009K-ND" x="86.2" y="11.5" size="1.778" layer="27" display="off"/>
+<attribute name="MF" value="Keystone" x="86.2" y="11.5" size="1.778" layer="27" display="off"/>
+<attribute name="MPN" value="5009" x="86.2" y="11.5" size="1.778" layer="27" display="off"/>
 </element>
 <element name="TP13" library="BreakoutBoard" package="TESTPOINT" value="TESTPOINT-YELLOW" x="5" y="52">
@@
 </signal>
 </signals>
-<errors>
-</errors>
 </board>
 </drawing>
